Commit message: adding plugin RGB-D Camera realsense D435

File: src/at1_description/urdf/_d435.urdf.xacro (robot description, xacro)
@@ -42,13 +42,13 @@
     </joint>
     <link name="${name}_bottom_screw_frame"/>
-    <joint name="camera_link_joint" type="fixed">
+    <joint name="${name}_link_joint" type="fixed">
       <origin xyz="${d435_mesh_x_offset} ${d435_cam_depth_py} ${d435_cam_depth_pz}" rpy="0 0 0"/>
       <parent link="${name}_bottom_screw_frame"/>
-      <child link="camera_link" />
+      <child link="${name}_link" />
     </joint>
-    <link name="camera_link">
+    <link name="${name}_link">
       <visual>
         <!-- the mesh origin is at front plate in between the two infrared camera axes -->
-        <origin xyz="0 0 0" rpy="1.75 0 1.75"/>
+        <origin xyz="${d435_zero_depth_to_glass + d435_glass_to_front} ${-d435_cam_depth_py} 0" rpy="${M_PI/2} 0 ${M_PI/2}"/>
         <geometry>
           <!-- <box size="${d435_cam_width} ${d435_cam_height} ${d435_cam_depth}"/> -->
@@ -57,5 +57,5 @@
       </visual>
       <collision>
-        <origin xyz="0.003 0.065 0.007" rpy="0 0 0"/>
+        <origin xyz="0 ${-d435_cam_depth_py} 0" rpy="0 0 0"/>
         <geometry>
           <box size="${d435_cam_depth} ${d435_cam_width} ${d435_cam_height}"/>
@@ -73,11 +73,11 @@
       <!-- camera depth joints and links -->
       <joint name="${name}_depth_joint" type="fixed">
-        <origin xyz="0.05 0.028 0.013" rpy="0 0 0"/>
-        <parent link="camera_link"/>
+        <origin xyz="0 0 0" rpy="0 0 0"/>
+        <parent link="${name}_link"/>
         <child link="${name}_depth_frame" />
       </joint>
       <link name="${name}_depth_frame"/>
       <joint name="${name}_depth_optical_joint" type="fixed">
-        <origin xyz="0 0 0" rpy="-1.57 0 -1.57" />
+        <origin xyz="0 0 0" rpy="${-M_PI/2} 0 ${-M_PI/2}" />
         <parent link="${name}_depth_frame" />
         <child link="${name}_depth_optical_frame" />
@@ -87,5 +87,5 @@
       <joint name="${name}_infra1_joint" type="fixed">
         <origin xyz="0 ${d435_cam_depth_to_infra1_offset} 0" rpy="0 0 0" />
-        <parent link="camera_link" />
+        <parent link="${name}_link" />
         <child link="${name}_infra1_frame" />
       </joint>
@@ -100,5 +100,5 @@
       <joint name="${name}_infra2_joint" type="fixed">
         <origin xyz="0 ${d435_cam_depth_to_infra2_offset} 0" rpy="0 0 0" />
-        <parent link="camera_link" />
+        <parent link="${name}_link" />
         <child link="${name}_infra2_frame" />
       </joint>
@@ -112,11 +112,11 @@
       <!-- camera color joints and links -->
       <joint name="${name}_color_joint" type="fixed">
-        <origin xyz="0 0.018 0.013" rpy="0 0 0" />
-        <parent link="camera_link" />
+        <origin xyz="0 ${d435_cam_depth_to_color_offset} 0" rpy="0 0 0" />
+        <parent link="${name}_link" />
         <child link="${name}_color_frame" />
       </joint>
       <link name="${name}_color_frame"/>
       <joint name="${name}_color_optical_joint" type="fixed">
-        <origin xyz="0 0 0" rpy="-1.57 0 -1.57" />
+        <origin xyz="0 0 0" rpy="${-M_PI/2} 0 ${-M_PI/2}" />
         <parent link="${name}_color_frame" />
         <child link="${name}_color_optical_frame" />
@@ -125,5 +125,5 @@
     </xacro:if>
     <xacro:if value="$(arg add_plug)">
-      <xacro:usb_plug parent="camera_link">
+      <xacro:usb_plug parent="${name}_link">
         <origin xyz="${d435_cam_mount_from_center_offset - 0.02095} ${-d435_cam_depth_py - 0.0353} 0" rpy="0 0 0"/>
       </xacro:usb_plug>

File: src/at1_description/urdf/_usb_plug.urdf.xacro (robot description, xacro)
@@ -12,7 +12,7 @@
       <xacro:insert_block name="origin" />
       <parent link="${parent}" />
-      <child link="camera_link" />
+      <child link="${name}_link" />
     </joint>
-    <link name="camera_link">
+    <link name="${name}_link">
       <visual>
         <!-- 0.044850 0.008000 0.018500 -->

File: src/at1_description/urdf/at1.xacro (robot description, xacro)
@@ -1,16 +1,18 @@
 <?xml version='1.0'?>
 <robot name="at1" xmlns:xacro="http://www.ros.org/wiki/xacro">
-  <!--xacro:property name="cameraSize" value="0.05"/>
-  <xacro:property name="cameraMass" value="0.1"/-->
+  <xacro:property name="cameraSize" value="0.05"/>
+  <xacro:property name="cameraMass" value="0.1"/>
   <xacro:include filename="$(find at1_description)/urdf/at1.gazebo" />
   <xacro:include filename="$(find at1_description)/urdf/materials.xacro" />
   <xacro:include filename="$(find at1_description)/urdf/macros.xacro" />
-  <xacro:include filename="$(find at1_description)/urdf/_d435.urdf.xacro" />
-  <xacro:include filename="$(find at1_description)/urdf/_d435_imu_modules.urdf.xacro" />
-  <xacro:include filename="$(find at1_description)/urdf/_d435i.urdf.xacro" />
-  <!--xacro:property name="r200_cam_rgb_px" value="0.05"/>
+  <!--xacro:include filename="$(find at1_description)/urdf/kh.gazebo.xacro" /-->
+  <!--xacro:include filename="$(find at1_description)/urdf/_d435.urdf.xacro">
+    <sensor_d435 parent="frnt_cam_lnk"></sensor_d435>
+  </xacro:include-->
+  <xacro:property name="r200_cam_rgb_px" value="0.05"/>
   <xacro:property name="r200_cam_rgb_py" value="0.018"/>
   <xacro:property name="r200_cam_rgb_pz" value="0.013"/>
-  <xacro:property name="r200_cam_depth_offset" value="0.01"/-->
+  <xacro:property name="r200_cam_depth_offset" value="0.01"/>
+  <link name="base_link"/>
   <link name='chassis'>
     <pose>0 0 0.1 0 0 0</pose>
@@ -80,4 +82,9 @@
     </visual>
   </link>
+  <joint name="base_joint" type="fixed">
+    <origin xyz="0 0 0" rpy="0 0 0"/>
+    <parent link="base_link"/>
+    <child link="chassis" />
+  </joint>
   <link name="left_wheel">
     <!--origin xyz="0.1 0.13 0.1" rpy="0 1.5707 1.5707"/-->
@@ -172,16 +179,35 @@
     </inertial>
   </link>
+  <!--link name="frnt_cam_lnk">
+    <visual>
+     <origin xyz="0.005 0.065 0.007" rpy="1.57 0 1.57"/>
+      <geometry>
+       <mesh filename="$(find at1_description)/meshes/d435.dae"/>
+      </geometry>
+    </visual>
+    <collision>
+      <origin xyz="0.005 0.065 0.007" rpy="1.57 0 1.57"/>
+      <geometry>
+       <mesh filename="$(find at1_description)/meshes/d435.dae"/>
+      </geometry>
+    </collision>
+  </link>
+  <joint name="3dcamera_joint" type="fixed">
+    <origin xyz="0.22 -0.07 0.04" rpy="0 0 0"/>
+    <parent link="chassis"/>
+    <child link="frnt_cam_lnk"/>
+  </joint-->
   <!-- Realsense -->
-  <!--link name="camera_link">
+  <link name="camera_link">
     <visual>
-     <origin xyz="0 0 0" rpy="1.57 0 1.57"/>
-      <geometry>
-       <mesh filename="$(find at1_description)/meshes/r200.dae"/>
+     <origin xyz="0.007 0.065 0.007" rpy="1.57 0 1.57"/>
+      <geometry>
+       <mesh filename="$(find at1_description)/meshes/d435.dae"/>
       </geometry>
     </visual>
     <collision>
-      <origin xyz="0.003 0.065 0.007" rpy="0 0 0"/>
-      <geometry>
-        <box size="0.012 0.132 0.020"/>
+      <origin xyz="0.007 0.065 0.007" rpy="1.57 0 1.57"/>
+      <geometry>
+       <mesh filename="$(find at1_description)/meshes/d435.dae"/>
       </geometry>
     </collision>
@@ -215,4 +241,4 @@
     <child link="camera_depth_optical_frame"/>
   </joint>
-  <link name="camera_depth_optical_frame"/-->
+  <link name="camera_depth_optical_frame"/>
 </robot>
